Commit message: basic implementation of multi robot spawn in launch file barista_two_robots.launch.py

File: xacro/barista_robot_model.urdf.xacro (robot description, xacro)
@@ -1,4 +1,5 @@
 <?xml version="1.0"?>
 <robot xmlns:xacro="http://www.ros.org/wiki/xacro" name="barista_bot">
+<xacro:property name="robot_name" value="$(arg robot_name)"/>
 <xacro:include filename="$(find barista_robot_description)/xacro/caster_wheel.xacro" />
 <xacro:include filename="$(find barista_robot_description)/xacro/cup_holder_tray.xacro" />
@@ -116,4 +117,5 @@
 <plugin name="barista_bot_joint_state" filename="libgazebo_ros_joint_state_publisher.so">
     <ros>
+        <namespace>/${robot_name}</namespace>
         <remapping>~/out:=joint_states</remapping>
     </ros>
@@ -126,4 +128,7 @@
 <gazebo>
     <plugin filename="libgazebo_ros_diff_drive.so" name="differential_drive_controller">
+        <ros>
+            <namespace>/${robot_name}</namespace>
+        </ros>
         <!-- wheels -->
         <left_joint>main_body_to_left_wheel_link_joint</left_joint>
@@ -173,5 +178,5 @@
             <plugin name="laser" filename="libgazebo_ros_ray_sensor.so">
             <ros>
-                <namespace>/barista_bot</namespace>
+                <namespace>/${robot_name}</namespace>
                 <remapping>~/out:=/scan</remapping>
             </ros>
